Commit message: Added parameters to urdf file. Not done.

File: my_rb1_description/urdf/my_rb1_robot.urdf (robot description, URDF)
Before this commit: robot rb1_robot, 7 links, 6 joints
Links:
- link base_link: mass None -> 20; geometry collision cylinder length=.3 radius=.25; visual cylinder length=.3 radius=.25
- link left_wheel: mass None -> 1.25; geometry collision cylinder length=.03 radius=.025; visual cylinder length=.03 radius=.025
- link right_wheel: mass None -> 1.25; geometry collision cylinder length=.3 radius=.25; visual cylinder length=.03 radius=.025
Joints:
- joint base_link_back_caster_joint: type  -> continuous
- joint base_link_front_caster_joint: type  -> continuous
- joint base_link_front_laser_joint: type  -> fixed
- joint base_link_left_wheel_joint: axis (none) -> 0 1 0; child (none) -> left_wheel; origin (none) -> xyz=0.0 -0.2 -0.15 rpy=0 0 0; parent (none) -> base_link; type  -> continuous
- joint base_link_plate_joint: child (none) -> base_footprint; origin (none) -> xyz=0 0 -0.15 rpy=0 0 0; parent (none) -> base_link; type  -> fixed
- joint base_link_right_wheel_joint: axis (none) -> 0 1 0; child (none) -> right_wheel; origin (none) -> xyz=0.0 0.2 -0.15 rpy=0 0 0; parent (none) -> base_link; type  -> continuous
